File: notastarboy.kicad_sch (KiCad schematic)
At the start: 7 parts, among them J1 Conn_01x04_Pin, J2 Conn_01x08_Pin, SW1 SW_Push, SW2 SW_Push, U1 XIAO-ESP32-C3-SMD, U2 DHT11

Commit message: I remade the schematic cuz i messed up net labels in the first one
Connections:
- net DHT11 DATA: now also R1.2; no longer U1.2 (D1)
- net SCL: now also J1.2 (Pin_2)
- net SDA: now also J1.1 (Pin_1)
- new net DHT11_DATA: U1.2 (D1)
- no-connect marks 0 -> 17
Changed lines of the file:
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@@
 	(generator_version "10.0")
 	(paper "A4")
+	(no_connect
+		(at 177.8 78.74)
+	)
+	(no_connect
+		(at 45.72 63.5)
+	)
+	(no_connect
+		(at 87.63 78.74)
+	)
+	(no_connect
+		(at 72.39 50.8)
+	)
+	(no_connect
+		(at 177.8 86.36)
+	)
+	(no_connect
+		(at 45.72 86.36)
+	)
+	(no_connect
+		(at 87.63 86.36)
+	)
+	(no_connect
+		(at 87.63 74.93)
+	)
+	(no_connect
+		(at 60.96 50.8)
+	)
+	(no_connect
+		(at 64.77 95.25)
+	)
+	(no_connect
+		(at 87.63 82.55)
+	)
+	(no_connect
+		(at 64.77 50.8)
+	)
+	(no_connect
+		(at 76.2 50.8)
+	)
+	(no_connect
+		(at 177.8 81.28)
+	)
+	(no_connect
+		(at 177.8 83.82)
+	)
+	(no_connect
+		(at 57.15 50.8)
+	)
+	(no_connect
+		(at 68.58 95.25)
+	)
 	(wire
 		(pts
@@
 	(wire
 		(pts
-			(xy 43.1785 78.74) (xy 45.72 78.74)
-		)
-		(stroke
-			(width 0)
-			(type default)
-		)
-	)
-	(wire
-		(pts
 			(xy 87.63 71.12) (xy 97.79 71.12)
 		)
@@
 	(wire
 		(pts
+			(xy 41.91 78.74) (xy 45.72 78.74)
+		)
+		(stroke
+			(width 0)
+			(type default)
+		)
+	)
+	(wire
+		(pts
 			(xy 176.53 48.26) (xy 176.53 49.53)
 		)
@@
 	(wire
 		(pts
-			(xy 130.81 104.14) (xy 135.89 104.14)
-		)
-		(stroke
-			(width 0)
-			(type default)
-		)
-	)
-	(wire
-		(pts
 			(xy 43.18 71.12) (xy 45.72 71.12)
 		)
@@
 	(wire
 		(pts
+			(xy 121.92 104.14) (xy 135.89 104.14)
+		)
+		(stroke
+			(width 0)
+			(type default)
+		)
+	)
+	(wire
+		(pts
 			(xy 135.89 85.09) (xy 135.89 87.63)
 		)
@@
 			(width 0)
 			(type default)
+		)
+	)
+	(label "SCL"
+		(at 41.91 78.74 0)
+		(effects
+			(font
+				(size 1.27 1.27)
+			)
+			(justify left bottom)
 		)
 	)
@@
 		)
 	)
-	(label "SDA"
-		(at 176.53 52.07 90)
-		(effects
-			(font
-				(size 1.27 1.27)
-			)
-			(justify left bottom)
-		)
-	)
-	(label "DHT11 DATA"
-		(at 132.08 72.39 0)
-		(effects
-			(font
-				(size 1.27 1.27)
-			)
-			(justify left bottom)
-		)
-	)
-	(label "DHT11 DATA"
-		(at 124.46 104.14 0)
-		(effects
-			(font
-				(size 1.27 1.27)
-			)
-			(justify left bottom)
-		)
-	)
-	(label "SCL"
-		(at 43.18 78.74 0)
-		(effects
-			(font
-				(size 1.27 1.27)
-			)
-			(justify left bottom)
-		)
-	)
-	(label "SCL"
-		(at 173.99 52.07 90)
-		(effects
-			(font
-				(size 1.27 1.27)
-			)
-			(justify left bottom)
-		)
-	)
 	(label "GPIO3"
 		(at 43.18 74.93 0)
@@
 	)
 	(label "SCL"
-		(at 179.07 73.66 0)
+		(at 173.99 49.53 270)
+		(effects
+			(font
+				(size 1.27 1.27)
+			)
+			(justify right bottom)
+		)
+	)
+	(label "DHT11_DATA"
+		(at 43.18 67.31 0)
+		(effects
+			(font
+				(size 1.27 1.27)
+			)
+			(justify left bottom)
+		)
+	)
+	(label "SDA"
+		(at 176.53 49.53 270)
+		(effects
+			(font
+				(size 1.27 1.27)
+			)
+			(justify right bottom)
+		)
+	)
+	(label "DHT11 DATA"
+		(at 121.92 104.14 0)
 		(effects
 			(font
@@
 		)
 	)
+	(label "SCL"
+		(at 179.07 73.66 0)
+		(effects
+			(font
+				(size 1.27 1.27)
+			)
+			(justify left bottom)
+		)
+	)
+	(label "SCL"
+		(at 41.91 78.74 0)
+		(effects
+			(font
+				(size 1.27 1.27)
+			)
+			(justify left bottom)
+		)
+	)
 	(label "DHT11 DATA"
-		(at 43.18 67.31 0)
+		(at 134.62 72.39 0)
+		(effects
+			(font
+				(size 1.27 1.27)
+			)
+			(justify left bottom)
+		)
+	)
+	(label "SDA"
+		(at 179.07 76.2 0)
 		(effects
 			(font
@@
 		(effects
 			(font
-				(size 1.27 1.27)
-			)
-			(justify left bottom)
-		)
-	)
-	(label "SDA"
-		(at 179.07 76.2 0)
-		(effects
-			(font

Commit message: cleaned up the schematic even more and hopefully its the final version
Connections:
- net GND: no longer U1.18 (GND)
- no-connect marks 17 -> 18
Changed lines of the file:
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@@
+	)
+	(no_connect
+		(at 68.58 50.8)
 	)
 	(no_connect
@@
 	(wire
 		(pts
-			(xy 68.58 50.8) (xy 68.58 45.72)
-		)
-		(stroke
-			(width 0)
-			(type default)
-		)
-	)
-	(wire
-		(pts
 			(xy 43.18 67.31) (xy 45.72 67.31)
 		)
@@
 		(pts
 			(xy 119.38 45.72) (xy 123.19 45.72)
-		)
-		(stroke
-			(width 0)
-			(type default)
-		)
-	)
-	(wire
-		(pts
-			(xy 67.31 45.72) (xy 68.58 45.72)
 		)
 		(stroke
@@
 	)
 	(symbol
-		(lib_id "power:GND")
-		(at 67.31 45.72 0)
-		(unit 1)
-		(body_style 1)
-		(exclude_from_sim no)
-		(in_bom yes)
-		(on_board yes)
-		(in_pos_files yes)
-		(dnp no)
-		(fields_autoplaced yes)
-		(property "Reference" "#PWR02"
-			(at 67.31 52.07 0)
-			(hide yes)
-			(show_name no)
-			(do_not_autoplace no)
-			(effects
-				(font
-					(size 1.27 1.27)
-				)
-			)
-		)
-		(property "Value" "GND"
-			(at 67.31 50.8 0)
-			(show_name no)
-			(do_not_autoplace no)
-			(effects
-				(font
-					(size 1.27 1.27)
-				)
-			)
-		)
-		(property "Footprint" ""
-			(at 67.31 45.72 0)
-			(hide yes)
-			(show_name no)
-			(do_not_autoplace no)
-			(effects
-				(font
-					(size 1.27 1.27)
-				)
-			)
-		)
-		(property "Datasheet" ""
-			(at 67.31 45.72 0)
-			(hide yes)
-			(show_name no)
-			(do_not_autoplace no)
-			(effects
-				(font
-					(size 1.27 1.27)
-				)
-			)
-		)
-		(property "Description" "Power symbol creates a global label with name \"GND\" , ground"
-			(at 67.31 45.72 0)
-			(hide yes)
-			(show_name no)
-			(do_not_autoplace no)
-			(effects
-				(font
-					(size 1.27 1.27)
-				)
-			)
-		)
-		(pin "1"
-		)
-		(instances
-			(project "notastarboy"
-				(path "/33f2e576-0c08-4472-974b-329ca185fcb3"
-					(reference "#PWR02")
-					(unit 1)
-				)
-			)
-		)
-	)
-	(symbol
 		(lib_id "power:+3.3V")
 		(at 135.89 85.09 0)
@@
 		(property "Value" "GND"
 			(at 92.71 72.39 0)
-			(show_name no)
-			(do_not_autoplace no)
+			(hide yes)
+			(show_name no)
+			(do_not_autoplace no)
